File: Schematics/IoT_pj_schematic.brd (EAGLE design)
At the start: 58.8 x 37.1 mm, 109 parts, among them J1 -, J6 -, J7 -, Q1 2N7002, Q2 SIA817, Q3 2N7002, Q5 2N7002DW-7-FNO_PAD, U1 D21G18, U2 SN74AVC4T774, U3 SARA-U201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

Commit message: Fix: LED 3 name to MQTT_Conn
Add: Shielding vias
Parts:
- renumbered LED3 to MQTT_CON
Routing:
- net GND: vias 68 -> 92
Changed lines of the file:
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@@
 <setting verticaltext="up"/>
 </settings>
-<grid distance="5" unitdist="mil" unit="mil" style="dots" multiple="1" display="yes" altdistance="5" altunitdist="mil" altunit="mil"/>
+<grid distance="100" unitdist="mil" unit="mil" style="dots" multiple="1" display="yes" altdistance="5" altunitdist="mil" altunit="mil"/>
 <layers>
 <layer number="1" name="Top" color="4" fill="1" visible="yes" active="yes"/>
@@
 <attribute name="VALUE" x="17.431" y="23.86" size="1.27" layer="27" rot="R270"/>
 </element>
-<element name="LED3" library="led" library_urn="urn:adsk.eagle:library:259" package="SML0603" package3d_urn="urn:adsk.eagle:package:15832/1" value="" x="14.224" y="18.161" smashed="yes" rot="R270">
-<attribute name="NAME" x="15.224" y="19.161" size="1.27" layer="25" rot="R270"/>
+<element name="MQTT_CON" library="led" library_urn="urn:adsk.eagle:library:259" package="SML0603" package3d_urn="urn:adsk.eagle:package:15832/1" value="" x="14.224" y="18.161" smashed="yes" rot="R270">
+<attribute name="NAME" x="14.716" y="19.034" size="0.254" layer="25" rot="R270"/>
 <attribute name="VALUE" x="12.224" y="19.161" size="1.27" layer="27" rot="R270"/>
 </element>
@@
 <wire x1="22.636" y1="3.967" x2="22.606" y2="3.937" width="0.19" layer="1"/>
 <via x="44.958" y="9.779" extent="1-16" drill="0.2"/>
+<via x="5.08" y="35.56" extent="1-16" drill="0.2"/>
+<via x="25.4" y="35.56" extent="1-16" drill="0.2"/>
+<via x="27.94" y="35.56" extent="1-16" drill="0.2"/>
+<via x="30.48" y="35.56" extent="1-16" drill="0.2"/>
+<via x="33.02" y="35.56" extent="1-16" drill="0.2"/>
+<via x="35.56" y="35.56" extent="1-16" drill="0.2"/>
+<via x="38.1" y="35.56" extent="1-16" drill="0.2"/>
+<via x="40.64" y="35.56" extent="1-16" drill="0.2"/>
+<via x="43.18" y="35.56" extent="1-16" drill="0.2"/>
+<via x="45.72" y="35.56" extent="1-16" drill="0.2"/>
+<via x="48.26" y="35.56" extent="1-16" drill="0.2"/>
+<via x="50.8" y="35.56" extent="1-16" drill="0.2"/>
+<via x="53.34" y="35.56" extent="1-16" drill="0.2"/>
+<via x="55.88" y="12.7" extent="1-16" drill="0.2"/>
+<via x="55.88" y="10.16" extent="1-16" drill="0.2"/>
+<via x="55.88" y="7.62" extent="1-16" drill="0.2"/>
+<via x="53.34" y="2.54" extent="1-16" drill="0.2"/>
+<via x="50.8" y="2.54" extent="1-16" drill="0.2"/>
+<via x="48.26" y="2.54" extent="1-16" drill="0.2"/>
+<via x="45.72" y="2.54" extent="1-16" drill="0.2"/>
+<via x="43.18" y="2.54" extent="1-16" drill="0.2"/>
+<via x="40.64" y="2.54" extent="1-16" drill="0.2"/>
+<via x="38.1" y="2.54" extent="1-16" drill="0.2"/>
+<via x="30.48" y="2.54" extent="1-16" drill="0.2"/>
 </signal>
 <signal name="PB02_AIN10">
@@
 </signal>
 <signal name="PA10_TCC0-W2">
-<contactref element="LED3" pad="C"/>
+<contactref element="MQTT_CON" pad="C"/>
 <contactref element="U1" pad="15"/>
 <contactref element="U7" pad="3"/>
@@
 </signal>
 <signal name="N$25">
-<contactref element="LED3" pad="A"/>
+<contactref element="MQTT_CON" pad="A"/>
 <contactref element="R4" pad="2"/>
 <wire x1="14.224" y1="17.411" x2="14.224" y2="16.325" width="0.19" layer="1"/>
